Commit message: slam_toolbox is used and map is generated

File: description/robot.urdf.xacro (robot description, xacro)
@@ -5,3 +5,4 @@
   <xacro:include filename="inertial_macros.xacro"/>
 <xacro:include filename="laser.xacro"/>
+<xacro:include filename="camera.xacro"/>
 </robot>

File: description/robot_core.xacro (robot description, xacro)
@@ -13,4 +13,11 @@
 	<!-- BASE LINK -->
 	<link name="base_link">
+	</link>
+	<joint name="base_footprint_joint" type="fixed">
+		<parent link="base_link"/>
+		<child link="base_footprint"/>
+		<origin xyz="0 0 0" rpy="0 0 0"/>
+	</joint>
+	<link name="base_footprint">
 	</link>
 	<!-- CHASSIS -->
